File: PiUPS/PiUPS.kicad_pcb (KiCad board)
At the start: 2 copper layers, 87.4 x 56 mm, 112 parts, among them J1 USB_C_Receptacle_USB2.0, J2 USB_B_Micro, J3 Screw_Terminal_01x02, J4 Raspberry_Pi_2_3, J5 USB_A, J6 Screw_Terminal_01x02, Q1 IRF7404, Q2 IRF7404, Q3 IRLML2803TRPBF, Q4 IRF7404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

Commit message: added new gerbers
Routing:
- net VSYS: track 89.6 -> 90.7 mm
- net GND: track 33.4 -> 33.2 mm, vias 197 -> 199
Other:
- board text added: "JLCJLCJLCJLC"
- board text added: "Raspberry PI UPS rev 0.5 by DDL JAN 2022"
- board text removed: "Raspberry PI UPS by DDL JAN 2022"
